File: NC7WZ17 Breakout/NC7WZ17 Breakout.sch (KiCad schematic (older format))
At the start: 4 parts, among them J1 Conn_01x03, J2 Conn_01x04, U1 NC7WZ17P6X

Commit message: 0.1uF capacitor value
Parts:
- C1: value C -> 0.1uF
Changed lines of the file:
@@
 P 3950 2300
 F 0 "C1" H 4128 2346 50  0000 L CNN
-F 1 "C" H 4128 2255 50  0000 L CNN
+F 1 "0.1uF" H 4128 2255 50  0000 L CNN
 F 2 "Capacitor_SMD:C_0603_1608Metric" H 3950 2300 50  0001 C CNN
 F 3 "~" H 3950 2300 50  0001 C CNN
